Commit message: Mejora de parámetros: min_turning_r

File: install/imiev/share/imiev/models/imiev/robot.xacro (robot description, xacro)
@@ -25,5 +25,5 @@
   <!-- wheel_xoff was 1.25. New geometry: rear=0, front=2.5 -->
   <!-- We will specify positions directly in macro calls or new properties -->
-  <xacro:property name="steer_limit"   value="0.6"/>
+  <xacro:property name="steer_limit"   value="0.51"/>
   <!-- SENSORES (Shifted +1.25 in X) -->
   <xacro:property name="camera_x" value="2.25"/>
@@ -157,5 +157,5 @@
       <axis xyz="0 0 1"/> <!-- Gira en Z -->
       <limit lower="${-steer_limit}" upper="${steer_limit}" effort="10000" velocity="5.0"/>
-      <dynamics damping="10.0" friction="10.0"/>
+      <dynamics damping="1.0" friction="1.0"/>
     </joint>
     <!-- Link de la rueda -->

Commit message: Revisión parámetros: ya gira bien

File: install/imiev/share/imiev/models/imiev/robot.xacro (robot description, xacro)
@@ -1,270 +1 @@
-<?xml version="1.0"?>
-<robot name="imiev" xmlns:xacro="http://www.ros.org/wiki/xacro">
-  <!-- ===================== -->
-  <!--   PROPIEDADES BASE    -->
-  <!-- ===================== -->
-  <xacro:property name="base_width" value="1.86"/>
-  <xacro:property name="base_length" value="3.56"/>
-  <xacro:property name="base_height" value="1.64"/>
-  <xacro:property name="base_mass" value="1080"/>
-  <!-- MATERIALS -->
-  <material name="grey">
-    <color rgba="0.5 0.5 0.5 1.0"/>
-  </material>
-  <material name="black">
-    <color rgba="0.0 0.0 0.0 1.0"/>
-  </material>
-  <material name="red">
-    <color rgba="1.0 0.0 0.0 1.0"/>
-  </material>
-  <!-- RUEDAS -->
-  <xacro:property name="wheel_radius" value="0.30"/>
-  <xacro:property name="wheel_width"  value="0.22"/>
-  <xacro:property name="wheel_ygap"   value="0.0"/>
-  <xacro:property name="wheel_zoff"   value="0.0"/>
-  <!-- wheel_xoff was 1.25. New geometry: rear=0, front=2.5 -->
-  <!-- We will specify positions directly in macro calls or new properties -->
-  <xacro:property name="steer_limit"   value="0.51"/>
-  <!-- SENSORES (Shifted +1.25 in X) -->
-  <xacro:property name="camera_x" value="2.25"/>
-  <xacro:property name="camera_y" value="0.00"/>
-  <xacro:property name="camera_z" value="1.70"/>
-  <xacro:property name="lidar_x" value="2.25"/>
-  <xacro:property name="lidar_y" value="0.00"/>
-  <xacro:property name="lidar_z" value="1.70"/>
-  <xacro:property name="imu_x" value="0.00"/>
-  <xacro:property name="imu_y" value="0.00"/>
-  <xacro:property name="imu_z" value="1.70"/>
-  <xacro:property name="gps_x" value="0.00"/>
-  <xacro:property name="gps_y" value="0.0"/>
-  <xacro:property name="gps_z" value="1.70"/>
-  <!-- ===================== -->
-  <!--     MACROS INERCIA    -->
-  <!-- ===================== -->
-  <xacro:macro name="box_inertia" params="m w h d">
-    <inertial>
-      <origin xyz="0 0 0" rpy="0 0 0"/>
-      <mass value="${m}"/>
-      <inertia ixx="${(m/12)*(h*h + d*d)}"
-               iyy="${(m/12)*(w*w + d*d)}"
-               izz="${(m/12)*(w*w + h*h)}"
-               ixy="0" ixz="0" iyz="0"/>
-    </inertial>
-  </xacro:macro>
-  <xacro:macro name="cylinder_inertia" params="m r h">
-    <inertial>
-      <origin xyz="0 0 0" rpy="0 0 0"/>
-      <mass value="${m}"/>
-      <inertia ixx="${(m/12)*(3*r*r + h*h)}"
-               iyy="${(m/12)*(3*r*r + h*h)}"
-               izz="${(m/2)*(r*r)}"
-               ixy="0" ixz="0" iyz="0"/>
-    </inertial>
-  </xacro:macro>
-<!-- ===================== -->
-  <!--    BASE FOOTPRINT     -->
-  <!-- ===================== -->
-  <link name="base_footprint"/>
-  <!-- ===================== -->
-  <!--       BODY LINK       -->
-  <!-- ===================== -->
-    <link name="base_link">
-    <visual>
-      <!-- Shifted origin +1.25 -->
-      <origin xyz="1.25 0 0.82" rpy="0 0 0"/>
-      <geometry>
-        <box size="${base_length} ${base_width} ${base_height}"/>
-      </geometry>
-      <material name="grey"/>
-    </visual>
-    <collision>
-        <geometry>
-          <box size="${base_length} ${base_width} ${base_height}"/>
-        </geometry>
-         <!-- Shifted origin +1.25 -->
-        <origin xyz="1.25 0.0 0.82" rpy="0 0 0"/>
-      </collision>
-    <xacro:box_inertia m="${base_mass}" w="${base_width}" h="${base_height}" d="${base_length}"/>
-  </link>
-  <joint name="base_joint" type="fixed">
-    <parent link="base_footprint"/>
-    <child link="base_link"/>
-    <origin xyz="0 0 0.3" rpy="0 0 0"/>
-  </joint>
-  <!-- ===================== -->
-  <!--        RUEDAS         -->
-  <!-- ===================== -->
-  <!-- ===================== -->
-  <!--   MACRO RUEDA TRASERA -->
-  <!-- ===================== -->
-  <xacro:macro name="rear_wheel" params="prefix x_pos y_reflect">
-    <link name="${prefix}_link">
-      <visual>
-        <origin xyz="0 0 0" rpy="${pi/2} 0 0"/>
-        <geometry>
-          <cylinder radius="${wheel_radius}" length="${wheel_width}"/>
-        </geometry>
-        <material name="black"/>
-      </visual>
-      <collision>
-        <origin xyz="0 0 0" rpy="${pi/2} 0 0"/>
-        <geometry>
-          <cylinder radius="${wheel_radius}" length="${wheel_width}"/>
-        </geometry>
-        <surface>
-          <friction>
-            <ode>
-              <mu>0.8</mu>
-              <mu2>1.2</mu2>
-              <fdir1>0 0 0</fdir1>
-            </ode>
-          </friction>
-        </surface>
-      </collision>
-      <xacro:cylinder_inertia m="15.0" r="${wheel_radius}" h="${wheel_width}"/>
-    </link>
-    <joint name="${prefix}_joint" type="continuous">
-      <parent link="base_link"/>
-      <child  link="${prefix}_link"/>
-      <!-- x_pos is passed directly -->
-      <origin xyz="${x_pos} ${y_reflect*(base_width/2 + wheel_ygap)} ${-wheel_zoff}" rpy="0 0 0"/>
-      <axis xyz="0 1 0"/>
-      <limit effort="10000" velocity="1000"/>
-      <dynamics damping="0.0" friction="0.0"/>
-    </joint>
-  </xacro:macro>
-  <!-- ===================== -->
-  <!--   MACRO RUEDA DELANTERA (DIRECCION) -->
-  <!-- ===================== -->
-  <xacro:macro name="front_wheel" params="prefix x_pos y_reflect">
-    <!-- Link de dirección (Steering Link / Mangueta) -->
-    <link name="${prefix}_steering_link">
-      <visual>
-        <geometry><cylinder radius="0.05" length="0.05"/></geometry>
-        <material name="blue"><color rgba="0 0 1 1"/></material>
-      </visual>
-      <inertial>
-        <mass value="1.0"/>
-        <inertia ixx="0.01" ixy="0" ixz="0" iyy="0.01" iyz="0" izz="0.01"/>
-      </inertial>
-    </link>
-    <!-- Joint de dirección (Revolute) -->
-    <joint name="${prefix}_steering_joint" type="revolute">
-      <parent link="base_link"/>
-      <child link="${prefix}_steering_link"/>
-      <!-- x_pos is passed directly -->
-      <origin xyz="${x_pos} ${y_reflect*(base_width/2 + wheel_ygap)} ${-wheel_zoff}" rpy="0 0 0"/>
-      <axis xyz="0 0 1"/> <!-- Gira en Z -->
-      <limit lower="${-steer_limit}" upper="${steer_limit}" effort="10000" velocity="5.0"/>
-      <dynamics damping="1.0" friction="1.0"/>
-    </joint>
-    <!-- Link de la rueda -->
-    <link name="${prefix}_link">
-      <visual>
-        <origin xyz="0 0 0" rpy="${pi/2} 0 0"/>
-        <geometry>
-          <cylinder radius="${wheel_radius}" length="${wheel_width}"/>
-        </geometry>
-        <material name="black"/>
-      </visual>
-      <collision>
-        <origin xyz="0 0 0" rpy="${pi/2} 0 0"/>
-        <geometry>
-          <cylinder radius="${wheel_radius}" length="${wheel_width}"/>
-        </geometry>
-         <surface>
-          <friction>
-            <ode>
-              <mu>0.8</mu>
-              <mu2>1.2</mu2>
-              <fdir1>0 0 0</fdir1>
-            </ode>
-          </friction>
-        </surface>
-      </collision>
-      <xacro:cylinder_inertia m="15.0" r="${wheel_radius}" h="${wheel_width}"/>
-    </link>
-    <!-- Joint de la rueda (Continuous) -->
-    <joint name="${prefix}_joint" type="continuous">
-      <parent link="${prefix}_steering_link"/>
-      <child  link="${prefix}_link"/>
-      <origin xyz="0 0 0" rpy="0 0 0"/>
-      <axis xyz="0 1 0"/> <!-- Gira en Y -->
-      <limit effort="10000" velocity="1000"/>
-      <dynamics damping="0.0" friction="0.05"/>
-    </joint>
-  </xacro:macro>
-  <!-- Instanciar ruedas -->
-  <!-- Traseras (Fijas) - AHORA EN X=0 (Eje Trasero) -->
-  <xacro:rear_wheel prefix="rear_left_wheel" x_pos="0.0" y_reflect="1"/>
-  <xacro:rear_wheel prefix="rear_right_wheel" x_pos="0.0" y_reflect="-1"/>
-  <!-- Delanteras (Ackermann) - AHORA EN X=2.5 (Distancia entre ejes) -->
-  <xacro:front_wheel prefix="front_left_wheel" x_pos="2.5"  y_reflect="1"/>
-  <xacro:front_wheel prefix="front_right_wheel" x_pos="2.5"  y_reflect="-1"/>
-  <!-- ===================== -->
-  <!--   SENSORES SEPARADOS  -->
-  <!-- ===================== -->
-  <!-- CAMERA MODULE -->
-  <xacro:macro name="camera_module" params="x y z r p yaw parent">
-    <link name="camera_link">
-      <visual>
-        <geometry><box size="0.05 0.05 0.05"/></geometry>
-        <material name="red"/>
-      </visual>
-    </link>
-    <joint name="camera_joint" type="fixed">
-      <parent link="${parent}"/>
-      <child  link="camera_link"/>
-      <origin xyz="${x} ${y} ${z}" rpy="${r} ${p} ${yaw}"/>
-    </joint>
-  </xacro:macro>
-  <!-- LIDAR MODULE -->
-  <xacro:macro name="lidar_module" params="x y z r p yaw parent">
-    <link name="lidar_link">
-      <visual>
-        <geometry><cylinder radius="0.04" length="0.06"/></geometry>
-        <material name="red"/>
-      </visual>
-    </link>
-    <joint name="lidar_joint" type="fixed">
-      <parent link="${parent}"/>
-      <child  link="lidar_link"/>
-      <origin xyz="${x} ${y} ${z}" rpy="${r} ${p} ${yaw}"/>
-    </joint>
-  </xacro:macro>
-  <!-- IMU MODULE -->
-  <xacro:macro name="imu_module" params="x y z r p yaw parent">
-    <link name="imu_link">
-      <visual>
-        <geometry><box size="0.04 0.04 0.04"/></geometry>
-        <material name="red"/>
-      </visual>
-    </link>
-    <joint name="imu_joint" type="fixed">
-      <parent link="${parent}"/>
-      <child  link="imu_link"/>
-      <origin xyz="${x} ${y} ${z}" rpy="${r} ${p} ${yaw}"/>
-    </joint>
-  </xacro:macro>
-  <!-- GPS MODULE -->
-  <xacro:macro name="gps_module" params="x y z r p yaw parent">
-    <link name="gps_link">
-      <visual>
-        <geometry><sphere radius="0.03"/></geometry>
-        <material name="red"/>
-      </visual>
-    </link>
-    <joint name="gps_joint" type="fixed">
-      <parent link="${parent}"/>
-      <child  link="gps_link"/>
-      <origin xyz="${x} ${y} ${z}" rpy="${r} ${p} ${yaw}"/>
-    </joint>
-  </xacro:macro>
-  <!-- Instantiate modules -->
-  <xacro:camera_module x="${camera_x}" y="${camera_y}" z="${camera_z}" r="0" p="0" yaw="0" parent="base_link"/>
-  <xacro:lidar_module  x="${lidar_x}"  y="${lidar_y}"  z="${lidar_z}"  r="0" p="0" yaw="0" parent="base_link"/>
-  <xacro:imu_module    x="${imu_x}"    y="${imu_y}"    z="${imu_z}"    r="0" p="0" yaw="0" parent="base_link"/>
-  <xacro:gps_module    x="${gps_x}"    y="${gps_y}"    z="${gps_z}"    r="0" p="0" yaw="0" parent="base_link"/>
-  <!-- ARCHIVOS ADICIONALES -->
-  <xacro:include filename="$(find imiev)/models/imiev/robot.gazebo" />
-</robot>
+/home/insia/simulador_ws/imiev/build/imiev/models/robot.xacro

File: src/imiev/models/robot.xacro (robot description, xacro)
@@ -25,16 +25,16 @@
   <!-- wheel_xoff was 1.25. New geometry: rear=0, front=2.5 -->
   <!-- We will specify positions directly in macro calls or new properties -->
-  <xacro:property name="steer_limit"   value="0.51"/>
-  <!-- SENSORES (Shifted +1.25 in X) -->
-  <xacro:property name="camera_x" value="2.25"/>
+  <xacro:property name="steer_limit"   value="0.9"/>
+  <!-- SENSORES -->
+  <xacro:property name="camera_x" value="1.70"/>
   <xacro:property name="camera_y" value="0.00"/>
-  <xacro:property name="camera_z" value="1.70"/>
-  <xacro:property name="lidar_x" value="2.25"/>
+  <xacro:property name="camera_z" value="1.80"/>
+  <xacro:property name="lidar_x" value="1.50"/>
   <xacro:property name="lidar_y" value="0.00"/>
-  <xacro:property name="lidar_z" value="1.70"/>
-  <xacro:property name="imu_x" value="0.00"/>
+  <xacro:property name="lidar_z" value="2.10"/>
+  <xacro:property name="imu_x" value="-1.00"/>
   <xacro:property name="imu_y" value="0.00"/>
   <xacro:property name="imu_z" value="1.70"/>
-  <xacro:property name="gps_x" value="0.00"/>
+  <xacro:property name="gps_x" value="-1.20"/>
   <xacro:property name="gps_y" value="0.0"/>
   <xacro:property name="gps_z" value="1.70"/>
@@ -72,5 +72,6 @@
     <visual>
       <!-- Shifted origin +1.25 -->
-      <origin xyz="1.25 0 0.82" rpy="0 0 0"/>
+      <!-- Shifted origin to center -->
+      <origin xyz="0 0 0.82" rpy="0 0 0"/>
       <geometry>
         <box size="${base_length} ${base_width} ${base_height}"/>
@@ -83,5 +84,6 @@
         </geometry>
          <!-- Shifted origin +1.25 -->
-        <origin xyz="1.25 0.0 0.82" rpy="0 0 0"/>
+         <!-- Shifted origin to center -->
+        <origin xyz="0 0 0.82" rpy="0 0 0"/>
       </collision>
     <xacro:box_inertia m="${base_mass}" w="${base_width}" h="${base_height}" d="${base_length}"/>
@@ -196,10 +198,10 @@
   </xacro:macro>
   <!-- Instanciar ruedas -->
-  <!-- Traseras (Fijas) - AHORA EN X=0 (Eje Trasero) -->
-  <xacro:rear_wheel prefix="rear_left_wheel" x_pos="0.0" y_reflect="1"/>
-  <xacro:rear_wheel prefix="rear_right_wheel" x_pos="0.0" y_reflect="-1"/>
-  <!-- Delanteras (Ackermann) - AHORA EN X=2.5 (Distancia entre ejes) -->
-  <xacro:front_wheel prefix="front_left_wheel" x_pos="2.5"  y_reflect="1"/>
-  <xacro:front_wheel prefix="front_right_wheel" x_pos="2.5"  y_reflect="-1"/>
+  <!-- Traseras (Fijas) - AHORA EN X=-1.25 -->
+  <xacro:rear_wheel prefix="rear_left_wheel" x_pos="-1.25" y_reflect="1"/>
+  <xacro:rear_wheel prefix="rear_right_wheel" x_pos="-1.25" y_reflect="-1"/>
+  <!-- Delanteras (Ackermann) - AHORA EN X=1.25 -->
+  <xacro:front_wheel prefix="front_left_wheel" x_pos="1.25"  y_reflect="1"/>
+  <xacro:front_wheel prefix="front_right_wheel" x_pos="1.25"  y_reflect="-1"/>
   <!-- ===================== -->
   <!--   SENSORES SEPARADOS  -->
